File: pcb/pcb.sch (KiCad schematic (older format))
At the start: 12 parts

Commit message: Update
Parts:
- IC1: renamed from IC?; footprint SOIC127P600X175-8N -> DS18B20Z+T&R:SOIC127P600X175-8N
- IC2: renamed from IC?; footprint DHT22 -> DHT22:DHT22
- gave numbers to parts that had none: 10
Connections:
- net labels removed: Anemometre, Girouette
Other:
- note added: "LiPo Rider"
Changed lines of the file:
@@
 $EndDescr
 $Comp
-L NUCLEO_L432KC:NUCLEO_L432KC L432KC?
+L NUCLEO_L432KC:NUCLEO_L432KC L432KC1
 U 1 1 5F98491B
 P 5450 3100
-F 0 "L432KC?" H 5850 3365 50  0000 C CNN
+F 0 "L432KC1" H 5850 3365 50  0000 C CNN
 F 1 "NUCLEO_L432KC" H 5850 3274 50  0000 C CNN
 F 2 "" H 5800 3350 50  0001 C CNN
@@
 	7050 3200 7050 3300
 $Comp
-L DS18B20Z+T&R:DS18B20Z+T&R IC?
+L DS18B20Z+T&R:DS18B20Z+T&R IC1
 U 1 1 5F98DE86
 P 2250 5950
-F 0 "IC?" H 2900 6215 50  0000 C CNN
+F 0 "IC1" H 2900 6215 50  0000 C CNN
 F 1 "DS18B20Z+T&R" H 2900 6124 50  0000 C CNN
-F 2 "SOIC127P600X175-8N" H 3400 6050 50  0001 L CNN
+F 2 "DS18B20Z+T&R:SOIC127P600X175-8N" H 3400 6050 50  0001 L CNN
 F 3 "https://datasheet.datasheetarchive.com/originals/dk/DKDS-25/482711.pdf" H 3400 5950 50  0001 L CNN
 F 4 "Board Mount Temperature Sensors Programmable Resolution 1-Wire Digital Thermometer" H 3400 5850 50  0001 L CNN "Description"
@@
 	3750 6250 3750 6350
 $Comp
-L Device:R R?
+L Device:R R1
 U 1 1 5F9928E6
 P 1900 6250
-F 0 "R?" V 1700 6200 50  0000 L CNN
+F 0 "R1" V 1700 6200 50  0000 L CNN
 F 1 "4.7k" V 1800 6200 50  0000 L CNN
 F 2 "" V 1830 6250 50  0001 C CNN
@@
 Sonde température DS18B20
 $Comp
-L DHT22:DHT22 IC?
+L DHT22:DHT22 IC2
 U 1 1 5F99F418
 P 5150 5950
-F 0 "IC?" H 5878 5846 50  0000 L CNN
+F 0 "IC2" H 5878 5846 50  0000 L CNN
 F 1 "DHT22" H 5878 5755 50  0000 L CNN
-F 2 "DHT22" H 5900 6050 50  0001 L CNN
+F 2 "DHT22:DHT22" H 5900 6050 50  0001 L CNN
 F 3 "https://datasheet4u.com/datasheet-parts/DHT22-datasheet.php?id=792211" H 5900 5950 50  0001 L CNN
 F 4 "Digital-output relative humidity & temperature sensor/module DHT22" H 5900 5850 50  0001 L CNN "Description"
@@
 Sonde température et humidité extérieure DHT22
 $Comp
-L Connector:AudioJack3 J?
+L Connector:AudioJack3 J3
 U 1 1 5FA07097
 P 8100 5300
-F 0 "J?" H 7821 5233 50  0000 R CNN
+F 0 "J3" H 7821 5233 50  0000 R CNN
 F 1 "AudioJack3" H 7821 5324 50  0000 R CNN
 F 2 "" H 8100 5300 50  0001 C CNN
@@
 $EndComp
 $Comp
-L Amplifier_Audio:LM386 U?
+L Amplifier_Audio:LM386 U1
 U 1 1 5FA08727
 P 9050 5300
-F 0 "U?" H 9394 5346 50  0000 L CNN
+F 0 "U1" H 9394 5346 50  0000 L CNN
 F 1 "LM386" H 9394 5255 50  0000 L CNN
 F 2 "" H 9150 5400 50  0001 C CNN
@@
 Text Label 8700 4950 0    50   ~ 0
 +5V
-Text Label 6500 3400 0    50   ~ 0
+Text Label 6650 3400 0    50   ~ 0
 +5V
-Text Label 6450 4400 0    50   ~ 0
+Text Label 6650 4400 0    50   ~ 0
 +3V3
 Wire Wire Line
@@
 Wire Wire Line
 	6350 3400 6650 3400
-Text Label 6550 4200 0    50   ~ 0
+Text Label 6650 4200 0    50   ~ 0
 A0
-Text Label 9700 5300 0    50   ~ 0
+Text Label 9800 5300 0    50   ~ 0
 A0
 Wire Notes Line
@@
 NoConn ~ 2250 5950
 $Comp
-L Conn_PHP2:Conn_PHP2 J?
+L Conn_PHP2:Conn_PHP2 J1
 U 1 1 5FA40DE7
 P 1100 1800
-F 0 "J?" H 1180 1792 50  0000 L CNN
+F 0 "J1" H 1180 1792 50  0000 L CNN
 F 1 "V_BAT" H 1180 1701 50  0000 L CNN
 F 2 "" H 1100 1800 50  0001 C CNN
@@
 Wire Wire Line
 	5350 3600 5050 3600
-Text Label 6500 4100 0    50   ~ 0
-Girouette
-Text Label 4800 3600 0    50   ~ 0
-Anemometre
-$Comp
-L Connector:4P4C J?
+$Comp
+L Connector:4P4C J4
 U 1 1 5FA2B8D0
 P 10550 1300
-F 0 "J?" H 10220 1396 50  0000 R CNN
+F 0 "J4" H 10220 1396 50  0000 R CNN
 F 1 "4P4C" H 10220 1305 50  0000 R CNN
 F 2 "" V 10550 1350 50  0001 C CNN
@@
 A1
 $Comp
-L Device:R R?
+L Device:R R3
 U 1 1 5FA320D9
 P 9700 1050
-F 0 "R?" H 9770 1096 50  0000 L CNN
+F 0 "R3" H 9770 1096 50  0000 L CNN
 F 1 "10k" H 9770 1005 50  0000 L CNN
 F 2 "" V 9630 1050 50  0001 C CNN
@@
 D3
 $Comp
-L Device:R R?
+L Device:R R4
 U 1 1 5FA36561
 P 9700 1750
-F 0 "R?" H 9770 1796 50  0000 L CNN
+F 0 "R4" H 9770 1796 50  0000 L CNN
 F 1 "10k" H 9770 1705 50  0000 L CNN
 F 2 "" V 9630 1750 50  0001 C CNN
@@
 Girouette et anémomètre
 $Comp
-L Device:R R?
+L Device:R R2
 U 1 1 5FA410B7
 P 4950 5900
-F 0 "R?" H 5020 5946 50  0000 L CNN
+F 0 "R2" H 5020 5946 50  0000 L CNN
 F 1 "1k" H 5020 5855 50  0000 L CNN
 F 2 "" V 4880 5900 50  0001 C CNN
@@
 Wire Wire Line
 	6350 3500 6650 3500
-Text Label 6550 3500 0    50   ~ 0
+Text Label 6650 3500 0    50   ~ 0
 A7
-Text Label 1400 1800 0    50   ~ 0
+Text Label 1500 1800 0    50   ~ 0
 A7
 $Comp
-L Conn_PHP2:Conn_PHP2 J?
+L Conn_PHP2:Conn_PHP2 J2
 U 1 1 5FA63282
 P 1100 2350
-F 0 "J?" H 1180 2342 50  0000 L CNN
+F 0 "J2" H 1180 2342 50  0000 L CNN
 F 1 "LIPO_OUT" H 1180 2251 50  0000 L CNN
 F 2 "" H 1100 2350 50  0001 C CNN
@@
 $EndComp
 $Comp
-L power:GND #PWR?
+L power:GND #PWR0106
 U 1 1 5FA637A2
 P 1300 2450
-F 0 "#PWR?" H 1300 2200 50  0001 C CNN
+F 0 "#PWR0106" H 1300 2200 50  0001 C CNN
 F 1 "GND" H 1305 2277 50  0000 C CNN
 F 2 "" H 1300 2450 50  0001 C CNN
@@
 Wire Wire Line
 	1300 2350 1500 2350
-Text Label 1350 2350 0    50   ~ 0
+Text Label 1500 2350 0    50   ~ 0
 +5V
+Text Label 5050 3600 0    50   ~ 0
+D3
+Text Label 6650 4100 0    50   ~ 0
+A1
+Wire Notes Line
+	650  1650 1850 1650
+Wire Notes Line
+	1850 1650 1850 2800
+Wire Notes Line
+	1850 2800 650  2800
+Wire Notes Line
+	650  2800 650  1650
+Text Notes 1050 1600 0    50   ~ 0
+LiPo Rider
 $EndSCHEMATC

Commit message: Finalisation PCB
Parts:
- removed IC1: DS18B20Z+T&R, DS18B20Z+T&R:SOIC127P600X175-8N, symbol DS18B20Z+T&R:DS18B20Z+T&R
- removed IC2: DHT22, DHT22:DHT22, symbol DHT22:DHT22
- removed J1: V_BAT, symbol Conn_PHP2:Conn_PHP2
- removed J2: LIPO_OUT, symbol Conn_PHP2:Conn_PHP2
- removed J4: 4P4C, symbol Connector:4P4C
- removed R4: 10k, symbol Device:R
- added C1: 1n, Capacitor_THT:CP_Radial_D4.0mm_P1.50mm, symbol Device:C
- added C2: 10u, Capacitor_THT:CP_Radial_D4.0mm_P1.50mm, symbol Device:C
- added C3: 1u, Capacitor_THT:CP_Radial_D4.0mm_P1.50mm, symbol Device:C
- added J1: VIN VBAT, Connector_PinHeader_2.00mm:PinHeader_1x04_P2.00mm_Vertical, symbol Connector_Generic:Conn_01x04
- added J2, J4, J6, J7: Conn_01x04, Connector_PinHeader_2.00mm:PinHeader_1x04_P2.00mm_Vertical, symbol Connector_Generic:Conn_01x04
- added J5: HX711, Connector_PinHeader_2.00mm:PinHeader_1x04_P2.00mm_Vertical, symbol Connector_Generic:Conn_01x04
- J3: footprint (none) -> Connector_Audio:Jack_3.5mm_Ledino_KB3SPRS_Horizontal
- L432KC1: footprint (none) -> NUCLEO-L432KC:MODULE_NUCLEO-L432KC
- R1, R3: footprint (none) -> Resistor_THT:R_Axial_DIN0204_L3.6mm_D1.6mm_P5.08mm_Horizontal
- R2: value 1k -> 10k; footprint (none) -> Resistor_THT:R_Axial_DIN0204_L3.6mm_D1.6mm_P5.08mm_Horizontal
- U1: footprint (none) -> LM386N-4_NOPB:DIP794W45P254L959H508Q8
Connections:
- net labels added: A2, A4
- net labels removed: A1
- no-connect marks 6 -> 5
Other:
- note added: "Capteur de poids"
- moved on the sheet: J3, U1

Commit message: Correction PCB + ajout module WISOL
Parts:
- added U2: WSSFM10R1AT, WSSFM10R1AT:XCVR_WSSFM10R1AT, symbol WSSFM10R1AT:WSSFM10R1AT
- C1: value 1n -> 1u; footprint Capacitor_THT:CP_Radial_D4.0mm_P1.50mm -> Capacitor_THT:CP_Radial_D5.0mm_P2.00mm
- C2: footprint Capacitor_THT:CP_Radial_D4.0mm_P1.50mm -> Capacitor_THT:CP_Radial_D5.0mm_P2.00mm
Connections:
- net +3V3: now also U2.21 (VDD_IO)
- net GND: now also U2.1 (GND), U2.2 (GND), U2.20 (GND), U2.22 (GND), U2.27 (GND), U2.28 (GND), U2.29 (GND), U2.3 (GND), U2.31 (GND), U2.4 (GND)
- net D1: now reaches L432KC1.PA9 (D1)
- net D1: now also U2.15 (UARTRX)
Other:
- note added: "Module Wisol Sigfox"
Changed lines of the file:
@@
 P 8850 5550
 F 0 "C1" V 8598 5550 50  0000 C CNN
-F 1 "1n" V 8689 5550 50  0000 C CNN
-F 2 "Capacitor_THT:CP_Radial_D4.0mm_P1.50mm" H 8888 5400 50  0001 C CNN
+F 1 "1u" V 8689 5550 50  0000 C CNN
+F 2 "Capacitor_THT:CP_Radial_D5.0mm_P2.00mm" H 8888 5400 50  0001 C CNN
 F 3 "~" H 8850 5550 50  0001 C CNN
 	1    8850 5550
@@
 F 0 "C2" V 8948 5100 50  0000 C CNN
 F 1 "10u" V 9039 5100 50  0000 C CNN
-F 2 "Capacitor_THT:CP_Radial_D4.0mm_P1.50mm" H 9238 4950 50  0001 C CNN
+F 2 "Capacitor_THT:CP_Radial_D5.0mm_P2.00mm" H 9238 4950 50  0001 C CNN
 F 3 "~" H 9200 5100 50  0001 C CNN
 	1    9200 5100
@@
 	1    0    0    -1
 $EndComp
+$Comp
+L WSSFM10R1AT:WSSFM10R1AT U2
+U 1 1 5FB95228
+P 2700 3900
+F 0 "U2" H 2700 4767 50  0000 C CNN
+F 1 "WSSFM10R1AT" H 2700 4676 50  0000 C CNN
+F 2 "WSSFM10R1AT:XCVR_WSSFM10R1AT" H 2700 3900 50  0001 L BNN
+F 3 "" H 2700 3900 50  0001 L BNN
+F 4 "WISOL" H 2700 3900 50  0001 L BNN "MANUFACTURER"
+	1    2700 3900
+	1    0    0    -1
+$EndComp
+$Comp
+L power:GND #PWR0117
+U 1 1 5FB961B3
+P 3500 4800
+F 0 "#PWR0117" H 3500 4550 50  0001 C CNN
+F 1 "GND" H 3505 4627 50  0000 C CNN
+F 2 "" H 3500 4800 50  0001 C CNN
+F 3 "" H 3500 4800 50  0001 C CNN
+	1    3500 4800
+	1    0    0    -1
+$EndComp
+Wire Wire Line
+	3500 3300 3750 3300
+Text Label 3750 3300 0    50   ~ 0
++3V3
+Wire Wire Line
+	5350 3100 5050 3100
+Text Label 5050 3100 0    50   ~ 0
+D1
+Wire Wire Line
+	1900 3400 1650 3400
+Text Label 1650 3400 0    50   ~ 0
+D1
+Wire Notes Line
+	4300 2900 4300 5050
+Wire Notes Line
+	4300 5050 1600 5050
+Wire Notes Line
+	1600 5050 1600 2900
+Wire Notes Line
+	1600 2900 4300 2900
+Text Notes 2550 2850 0    50   ~ 0
+Module Wisol Sigfox
 $EndSCHEMATC

Commit message: Finalisation PCB
Parts:
- removed U2: WSSFM10R1AT, WSSFM10R1AT:XCVR_WSSFM10R1AT, symbol WSSFM10R1AT:WSSFM10R1AT
- added J8: Conn_01x08, Connector_PinHeader_2.00mm:PinHeader_1x08_P2.00mm_Vertical, symbol Connector_Generic:Conn_01x08
- added R4: 2k, Resistor_THT:R_Axial_DIN0204_L3.6mm_D1.6mm_P5.08mm_Vertical, symbol Device:R
- added R5: 1k, Resistor_THT:R_Axial_DIN0204_L3.6mm_D1.6mm_P5.08mm_Vertical, symbol Device:R
Connections:
- net +3V3: now also J8.2 (Pin_2)
- net A7: now also R4.2, R5.1; no longer J1.1 (Pin_1)
- net D1: now also J8.8 (Pin_8)
- net GND: now also J8.1 (Pin_1), R5.2
- new net: J1.1 (Pin_1), R4.1
Changed lines of the file:
@@
 Text Label 6650 3500 0    50   ~ 0
-A7
-Text Label 1400 2250 0    50   ~ 0
 A7
 $Comp
@@
 Text Label 5050 3600 0    50   ~ 0
 D3
-Wire Notes Line
-	1850 1650 1850 2800
-Wire Notes Line
-	1850 2800 650  2800
 Wire Notes Line
 	650  2800 650  1650
@@
 $EndComp
 NoConn ~ 1200 2350
-Wire Notes Line
-	1850 1650 650  1650
 $Comp
 L Device:R R1
@@
 $EndComp
 $Comp
-L WSSFM10R1AT:WSSFM10R1AT U2
-U 1 1 5FB95228
-P 2700 3900
-F 0 "U2" H 2700 4767 50  0000 C CNN
-F 1 "WSSFM10R1AT" H 2700 4676 50  0000 C CNN
-F 2 "WSSFM10R1AT:XCVR_WSSFM10R1AT" H 2700 3900 50  0001 L BNN
-F 3 "" H 2700 3900 50  0001 L BNN
-F 4 "WISOL" H 2700 3900 50  0001 L BNN "MANUFACTURER"
-	1    2700 3900
-	1    0    0    -1
-$EndComp
-$Comp
 L power:GND #PWR0117
 U 1 1 5FB961B3
-P 3500 4800
-F 0 "#PWR0117" H 3500 4550 50  0001 C CNN
-F 1 "GND" H 3505 4627 50  0000 C CNN
-F 2 "" H 3500 4800 50  0001 C CNN
-F 3 "" H 3500 4800 50  0001 C CNN
-	1    3500 4800
-	1    0    0    -1
-$EndComp
-Wire Wire Line
-	3500 3300 3750 3300
-Text Label 3750 3300 0    50   ~ 0
+P 2500 4250
+F 0 "#PWR0117" H 2500 4000 50  0001 C CNN
+F 1 "GND" H 2505 4077 50  0000 C CNN
+F 2 "" H 2500 4250 50  0001 C CNN
+F 3 "" H 2500 4250 50  0001 C CNN
+	1    2500 4250
+	1    0    0    -1
+$EndComp
+Wire Wire Line
+	2500 4150 2750 4150
+Text Label 2750 4150 0    50   ~ 0
 +3V3
 Wire Wire Line
@@
 D1
 Wire Wire Line
-	1900 3400 1650 3400
-Text Label 1650 3400 0    50   ~ 0
+	2500 3550 2750 3550
+Text Label 2750 3550 2    50   ~ 0
 D1
 Wire Notes Line
@@
 Text Notes 2550 2850 0    50   ~ 0
 Module Wisol Sigfox
+$Comp
+L Device:R R4
+U 1 1 5FBBD368
+P 1800 2100
+F 0 "R4" H 1870 2146 50  0000 L CNN
+F 1 "2k" H 1870 2055 50  0000 L CNN
+F 2 "Resistor_THT:R_Axial_DIN0204_L3.6mm_D1.6mm_P5.08mm_Vertical" V 1730 2100 50  0001 C CNN
+F 3 "~" H 1800 2100 50  0001 C CNN
+	1    1800 2100
+	1    0    0    -1
+$EndComp
+$Comp
+L Device:R R5
+U 1 1 5FBBD807
+P 1800 2400
+F 0 "R5" H 1870 2446 50  0000 L CNN
+F 1 "1k" H 1870 2355 50  0000 L CNN
+F 2 "Resistor_THT:R_Axial_DIN0204_L3.6mm_D1.6mm_P5.08mm_Vertical" V 1730 2400 50  0001 C CNN
+F 3 "~" H 1800 2400 50  0001 C CNN
+	1    1800 2400
+	1    0    0    -1
+$EndComp
+$Comp
+L power:GND #PWR0118
+U 1 1 5FBBDDB8
+P 1800 2550
+F 0 "#PWR0118" H 1800 2300 50  0001 C CNN
+F 1 "GND" H 1805 2377 50  0000 C CNN
+F 2 "" H 1800 2550 50  0001 C CNN
+F 3 "" H 1800 2550 50  0001 C CNN
+	1    1800 2550
+	1    0    0    -1
+$EndComp
+Wire Wire Line
+	1400 2250 1400 1950
+Wire Wire Line
+	1400 1950 1800 1950
+Wire Wire Line
+	1800 2250 2100 2250
+Connection ~ 1800 2250
+Text Label 2100 2250 0    50   ~ 0
+A7
+Wire Notes Line
+	2250 2800 2250 1650
+Wire Notes Line
+	650  2800 2250 2800
+Wire Notes Line
+	650  1650 2250 1650
+$Comp
+L Connector_Generic:Conn_01x08 J8
+U 1 1 5FBC63C9
+P 2300 3950
+F 0 "J8" H 2218 3325 50  0000 C CNN
+F 1 "Conn_01x08" H 2218 3416 50  0000 C CNN
+F 2 "Connector_PinHeader_2.00mm:PinHeader_1x08_P2.00mm_Vertical" H 2300 3950 50  0001 C CNN
+F 3 "~" H 2300 3950 50  0001 C CNN
+	1    2300 3950
+	-1   0    0    1
+$EndComp
 $EndSCHEMATC

Commit message: ...
Parts:
- R4: value 2k -> 1K
- R5: value 1k -> 2k
Connections:
- net GND: now also J6.2 (Pin_2)
- no-connect marks 5 -> 4
Changed lines of the file:
@@
 D3
 NoConn ~ 10650 1700
-NoConn ~ 10650 1050
 $Comp
 L Connector_Generic:Conn_01x04 J1
@@
 P 1800 2100
 F 0 "R4" H 1870 2146 50  0000 L CNN
-F 1 "2k" H 1870 2055 50  0000 L CNN
+F 1 "1K" H 1870 2055 50  0000 L CNN
 F 2 "Resistor_THT:R_Axial_DIN0204_L3.6mm_D1.6mm_P5.08mm_Vertical" V 1730 2100 50  0001 C CNN
 F 3 "~" H 1800 2100 50  0001 C CNN
@@
 P 1800 2400
 F 0 "R5" H 1870 2446 50  0000 L CNN
-F 1 "1k" H 1870 2355 50  0000 L CNN
+F 1 "2k" H 1870 2355 50  0000 L CNN
 F 2 "Resistor_THT:R_Axial_DIN0204_L3.6mm_D1.6mm_P5.08mm_Vertical" V 1730 2400 50  0001 C CNN
 F 3 "~" H 1800 2400 50  0001 C CNN
@@
 	-1   0    0    1
 $EndComp
+$Comp
+L power:GND #PWR0119
+U 1 1 5FBD8442
+P 10650 1050
+F 0 "#PWR0119" H 10650 800 50  0001 C CNN
+F 1 "GND" H 10655 877 50  0000 C CNN
+F 2 "" H 10650 1050 50  0001 C CNN
+F 3 "" H 10650 1050 50  0001 C CNN
+	1    10650 1050
+	1    0    0    -1
+$EndComp
 $EndSCHEMATC

Commit message: Ajout choix alimentation
Parts:
- added SW1: SW_DPDT_x2, Button_Switch_SMD:SW_SPDT_CK-JS102011SAQN, symbol Switch:SW_DPDT_x2
- added U2: IFX27001TFV33, Package_TO_SOT_SMD:TO-252-3_TabPin2, symbol Regulator_Linear:IFX27001TFV33
Connections:
- net +3V3: now also U2.2 (Q)
- net +5V: now also SW1.1 (A); no longer J1.3 (Pin_3)
- net GND: now also U2.1 (GND)
- net D0: now reaches L432KC1.PA10 (D0)
- net D0: now also J8.7 (Pin_7)
- new net: SW1.3 (C), U2.3 (I)
- new net V_alim: J1.3 (Pin_3), SW1.2 (B)
Other:
- note added: "Choix tension d'alim"
- moved on the sheet: J8
Changed lines of the file:
@@
 Wire Wire Line
 	1200 2450 1400 2450
-Text Label 1400 2450 0    50   ~ 0
-+5V
 Text Label 5050 3600 0    50   ~ 0
 D3
@@
 L power:GND #PWR0117
 U 1 1 5FB961B3
-P 2500 4250
-F 0 "#PWR0117" H 2500 4000 50  0001 C CNN
-F 1 "GND" H 2505 4077 50  0000 C CNN
-F 2 "" H 2500 4250 50  0001 C CNN
-F 3 "" H 2500 4250 50  0001 C CNN
-	1    2500 4250
-	1    0    0    -1
-$EndComp
-Wire Wire Line
-	2500 4150 2750 4150
-Text Label 2750 4150 0    50   ~ 0
+P 2100 4750
+F 0 "#PWR0117" H 2100 4500 50  0001 C CNN
+F 1 "GND" H 2105 4577 50  0000 C CNN
+F 2 "" H 2100 4750 50  0001 C CNN
+F 3 "" H 2100 4750 50  0001 C CNN
+	1    2100 4750
+	1    0    0    -1
+$EndComp
+Wire Wire Line
+	2100 4650 2350 4650
+Text Label 2350 4650 2    50   ~ 0
 +3V3
 Wire Wire Line
@@
 D1
 Wire Wire Line
-	2500 3550 2750 3550
-Text Label 2750 3550 2    50   ~ 0
+	2100 4050 2350 4050
+Text Label 2350 4050 2    50   ~ 0
 D1
-Wire Notes Line
-	4300 2900 4300 5050
-Wire Notes Line
-	4300 5050 1600 5050
-Wire Notes Line
-	1600 5050 1600 2900
-Wire Notes Line
-	1600 2900 4300 2900
-Text Notes 2550 2850 0    50   ~ 0
-Module Wisol Sigfox
 $Comp
 L Device:R R4
@@
 L Connector_Generic:Conn_01x08 J8
 U 1 1 5FBC63C9
-P 2300 3950
-F 0 "J8" H 2218 3325 50  0000 C CNN
-F 1 "Conn_01x08" H 2218 3416 50  0000 C CNN
-F 2 "Connector_PinHeader_2.00mm:PinHeader_1x08_P2.00mm_Vertical" H 2300 3950 50  0001 C CNN
-F 3 "~" H 2300 3950 50  0001 C CNN
-	1    2300 3950
+P 1900 4450
+F 0 "J8" H 1818 3825 50  0000 C CNN
+F 1 "Conn_01x08" H 1818 3916 50  0000 C CNN
+F 2 "Connector_PinHeader_2.00mm:PinHeader_1x08_P2.00mm_Vertical" H 1900 4450 50  0001 C CNN
+F 3 "~" H 1900 4450 50  0001 C CNN
+	1    1900 4450
 	-1   0    0    1
 $EndComp
@@
 	1    0    0    -1
 $EndComp
+Wire Wire Line
+	2100 4150 2350 4150
+Wire Wire Line
+	5350 3200 5050 3200
+Text Label 5050 3200 0    50   ~ 0
+D0
+Text Label 2350 4150 2    50   ~ 0
+D0
+Text Notes 1650 3650 0    50   ~ 0
+Module Wisol Sigfox
+Wire Notes Line
+	1550 3700 2550 3700
+Wire Notes Line
+	2550 3700 2550 5050
+Wire Notes Line
+	2550 5050 1550 5050
+Wire Notes Line
+	1550 5050 1550 3700
+Text Label 1400 2450 0    50   ~ 0
+V_alim
+$Comp
+L Switch:SW_DPDT_x2 SW1
+U 1 1 5FBD3E89
+P 3300 2650
+F 0 "SW1" H 3300 2935 50  0000 C CNN
+F 1 "SW_DPDT_x2" H 3300 2844 50  0000 C CNN
+F 2 "Button_Switch_SMD:SW_SPDT_CK-JS102011SAQN" H 3300 2650 50  0001 C CNN
+F 3 "~" H 3300 2650 50  0001 C CNN
+	1    3300 2650
+	1    0    0    -1
+$EndComp
+Wire Wire Line
+	3100 2650 2850 2650
+Text Label 2850 2650 0    50   ~ 0
+V_alim
+$Comp
+L Regulator_Linear:IFX27001TFV33 U2
+U 1 1 5FBD8709
+P 3800 2750
+F 0 "U2" H 4100 2400 50  0000 C CNN
+F 1 "IFX27001TFV33" H 4150 2500 50  0000 C CNN
+F 2 "Package_TO_SOT_SMD:TO-252-3_TabPin2" H 3800 2700 50  0001 C CNN
+F 3 "https://static6.arrow.com/aropdfconversion/dc75757ae45a88e5f69bdce3f2a651a5fe0ca07d/ifx27001_ds_10.pdf" H 3800 2700 50  0001 C CNN
+	1    3800 2750
+	1    0    0    -1
+$EndComp
+$Comp
+L power:GND #PWR0120
+U 1 1 5FBD95A5
+P 3800 3050
+F 0 "#PWR0120" H 3800 2800 50  0001 C CNN
+F 1 "GND" H 3805 2877 50  0000 C CNN
+F 2 "" H 3800 3050 50  0001 C CNN
+F 3 "" H 3800 3050 50  0001 C CNN
+	1    3800 3050
+	1    0    0    -1
+$EndComp
+Wire Wire Line
+	3500 2550 4250 2550
+Wire Wire Line
+	4100 2750 4250 2750
+Text Label 4250 2550 0    50   ~ 0
++5V
+Text Label 4250 2750 0    50   ~ 0
++3V3
+Wire Notes Line
+	2750 2250 4600 2250
+Wire Notes Line
+	4600 2250 4600 3350
+Wire Notes Line
+	4600 3350 2750 3350
+Wire Notes Line
+	2750 3350 2750 2250
+Text Notes 3300 2200 0    50   ~ 0
+Choix tension d'alim
 $EndSCHEMATC
