File: pcb/_autosave-pcb.sch (KiCad schematic (older format))
At the start: 22 parts, among them J1 VIN VBAT, J2 Conn_01x04, J3 AudioJack3, J4 Conn_01x04, J5 HX711, J6 Conn_01x04, J7 Conn_01x04, J8 Conn_01x08, SW1 SW_DPDT_x2, U1 LM386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

Commit message: Finalisation PCB
Parts:
- C4, C5: renamed from C?; footprint (none) -> Capacitor_SMD:C_0805_2012Metric_Pad1.18x1.45mm_HandSolder
Changed lines of the file:
@@
 $EndComp
 $Comp
-L Device:C C?
+L Device:C C4
 U 1 1 5FBFE6BC
 P 4300 3000
-F 0 "C?" H 4200 3100 50  0000 L CNN
+F 0 "C4" H 4200 3100 50  0000 L CNN
 F 1 "470p" H 4150 2900 50  0000 L CNN
-F 2 "" H 4338 2850 50  0001 C CNN
+F 2 "Capacitor_SMD:C_0805_2012Metric_Pad1.18x1.45mm_HandSolder" H 4338 2850 50  0001 C CNN
 F 3 "~" H 4300 3000 50  0001 C CNN
 	1    4300 3000
@@
 $EndComp
 $Comp
-L power:GND #PWR?
+L power:GND #PWR0122
 U 1 1 5FBFF114
 P 4300 3150
-F 0 "#PWR?" H 4300 2900 50  0001 C CNN
+F 0 "#PWR0122" H 4300 2900 50  0001 C CNN
 F 1 "GND" H 4305 2977 50  0000 C CNN
 F 2 "" H 4300 3150 50  0001 C CNN
@@
 	4300 2850 4200 2850
 $Comp
-L Device:C C?
+L Device:C C5
 U 1 1 5FC01AAB
 P 4550 3000
-F 0 "C?" H 4665 3046 50  0000 L CNN
+F 0 "C5" H 4665 3046 50  0000 L CNN
 F 1 "2.2u" H 4665 2955 50  0000 L CNN
-F 2 "" H 4588 2850 50  0001 C CNN
+F 2 "Capacitor_SMD:C_0805_2012Metric_Pad1.18x1.45mm_HandSolder" H 4588 2850 50  0001 C CNN
 F 3 "~" H 4550 3000 50  0001 C CNN
 	1    4550 3000
@@
 	4200 2750 4550 2750
 $Comp
-L power:GND #PWR?
+L power:GND #PWR0123
 U 1 1 5FC05656
 P 4550 3150
-F 0 "#PWR?" H 4550 2900 50  0001 C CNN
+F 0 "#PWR0123" H 4550 2900 50  0001 C CNN
 F 1 "GND" H 4555 2977 50  0000 C CNN
 F 2 "" H 4550 3150 50  0001 C CNN
