File: pcb/_autosave-pcb.sch (KiCad schematic (older format))
At the start: 22 parts, among them J1 VIN VBAT, J2 Conn_01x04, J3 AudioJack3, J4 Conn_01x04, J5 Conn_01x05, J6 Conn_01x04, J7 Conn_01x04, J8 Conn_01x08, SW1 SW_DPDT_x2, U1 LM386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

Commit message: Ajout via
Parts:
- R4: value 1K -> 2.2k
- R5: value 2k -> 3.3k
Connections:
- net D10: now reaches L432KC1.PA11 (D10)
- net D10: now also J2.1 (Pin_1)
- net CLK: now reaches L432KC1.PA7 (A6)
- net CLK: now also J5.4 (Pin_4)
- net A1: no longer names the net of L432KC1.PA1 (A1)
- net A1: no longer J5.3 (Pin_3)
- net A2: no longer names the net of L432KC1.PA3 (A2)
- net A2: no longer J5.4 (Pin_4)
- net D12 renamed DATA
- net DATA: now also J5.3 (Pin_3); no longer J2.1 (Pin_1)
Changed lines of the file:
@@
 	7050 3200 7050 3300
 Wire Wire Line
-	5350 4500 5050 4500
-Text Label 5050 4500 0    50   ~ 0
-D12
+	5350 4300 5050 4300
 Wire Notes Line
 	1000 5600 3950 5600
@@
 Text Label 5800 1150 0    50   ~ 0
 +3V3
-Wire Wire Line
-	6350 4000 6650 4000
-Text Label 6650 4000 0    50   ~ 0
-A2
 $Comp
 L Connector_Generic:Conn_01x04 J2
@@
 Wire Wire Line
 	2700 6300 2350 6300
-Text Label 2350 6100 0    50   ~ 0
-D12
 Text Label 2350 6300 0    50   ~ 0
 +3V3
@@
 Text Label 10200 1150 0    50   ~ 0
 +5V
-Text Label 10200 950  0    50   ~ 0
-A4
 Text Label 10200 1800 0    50   ~ 0
 +5V
@@
 $EndComp
 Wire Wire Line
-	6350 3800 6650 3800
-Text Label 6650 3800 0    50   ~ 0
-A4
-Wire Wire Line
 	9500 5350 9500 5250
 Wire Wire Line
@@
 P 1800 2100
 F 0 "R4" H 1870 2146 50  0000 L CNN
-F 1 "1K" H 1870 2055 50  0000 L CNN
+F 1 "2.2k" H 1870 2055 50  0000 L CNN
 F 2 "Resistor_THT:R_Axial_DIN0207_L6.3mm_D2.5mm_P10.16mm_Horizontal" V 1730 2100 50  0001 C CNN
 F 3 "~" H 1800 2100 50  0001 C CNN
@@
 P 1800 2400
 F 0 "R5" H 1870 2446 50  0000 L CNN
-F 1 "2k" H 1870 2355 50  0000 L CNN
+F 1 "3.3k" H 1870 2355 50  0000 L CNN
 F 2 "Resistor_THT:R_Axial_DIN0207_L6.3mm_D2.5mm_P10.16mm_Horizontal" V 1730 2400 50  0001 C CNN
 F 3 "~" H 1800 2400 50  0001 C CNN
@@
 	6300 1250 6300 1150
 Connection ~ 6300 1150
-Wire Wire Line
-	6350 4100 6650 4100
-Text Label 6650 4100 0    50   ~ 0
-A1
+Text Label 6000 1450 0    50   ~ 0
+CLK
 Text Label 6000 1350 0    50   ~ 0
-A1
-Text Label 6000 1450 0    50   ~ 0
-A2
+DATA
+Text Label 2350 6100 0    50   ~ 0
+D10
+Text Label 5050 4300 0    50   ~ 0
+D10
+Text Label 10200 950  0    50   ~ 0
+A4
+Text Label 6650 3800 0    50   ~ 0
+A4
+Wire Wire Line
+	6350 3800 6650 3800
+Wire Wire Line
+	6350 3600 6650 3600
+Text Label 6650 3600 0    50   ~ 0
+CLK
+Wire Wire Line
+	5350 4500 5050 4500
+Text Label 5050 4500 0    50   ~ 0
+DATA
 $EndSCHEMATC
