File: pcb/_autosave-pcb.kicad_pcb (KiCad board)
At the start: 2 copper layers, 22 parts, among them J1 VIN VBAT, J2 Conn_01x04, J3 AudioJack3, J4 Conn_01x04, J5 HX711, J6 Conn_01x04, J7 Conn_01x04, J8 Conn_01x08, SW1 SW_DPDT_x2, U1 LM386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

Commit message: Décalage pin header HX711
Parts:
- moved J5 1.00 mm to (176.0, 83.0)
Routing:
- net GND: track 20.5 -> 3.14 mm
- net /+3V3: track 201.2 -> 202.6 mm
Changed lines of the file:
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@@
     (thickness 1.6)
     (drawings 11)
-    (tracks 125)
+    (tracks 122)
     (zones 0)
     (modules 22)
@@
   )
   (module Connector_PinHeader_2.54mm:PinHeader_1x04_P2.54mm_Vertical (layer F.Cu)
-    (at 175 83 270)
+    (at 176 83 270)
     (descr "Through hole straight pin header, 1x04, 2.54mm pitch, single row")
     (tags "Through hole pin header THT 1x04 2.54mm single row")
@@
   (gr_line (start 184 55) (end 160 55) (layer F.CrtYd) (width 0.05))
   (segment (start 155 59.8625) (end 155 63) (width 0.4) (layer B.Cu) (net 1))
-  (segment (start 143.28 72.415) (end 136.585 72.415) (width 1.02) (layer F.Cu) (net 1))
-  (segment (start 131.505 77.495) (end 128.04 77.495) (width 1.02) (layer F.Cu) (net 1))
-  (segment (start 136.585 72.415) (end 131.505 77.495) (width 1.02) (layer F.Cu) (net 1))
   (segment (start 121.28 86.28) (end 123 86.28) (width 1.02) (layer B.Cu) (net 2))
   (segment (start 119 84) (end 121.28 86.28) (width 1.02) (layer B.Cu) (net 2))
@@
   (segment (start 121 98) (end 122 97) (width 1.02) (layer B.Cu) (net 5))
   (segment (start 154.9625 65) (end 154.9625 65.9625) (width 0.81) (layer B.Cu) (net 5))
+  (segment (start 156 67) (end 161 67) (width 0.81) (layer B.Cu) (net 5))
   (segment (start 154.9625 65.9625) (end 156 67) (width 0.81) (layer B.Cu) (net 5))
-  (segment (start 156 67) (end 161 67) (width 0.81) (layer B.Cu) (net 5))
-  (segment (start 175 81) (end 175 83) (width 0.81) (layer B.Cu) (net 5))
-  (segment (start 161 67) (end 175 81) (width 0.81) (layer B.Cu) (net 5))
   (segment (start 147.895 102.895) (end 149 104) (width 1.02) (layer B.Cu) (net 5))
   (segment (start 143.28 102.895) (end 147.895 102.895) (width 1.02) (layer B.Cu) (net 5))
@@
   (segment (start 172 103) (end 169 103) (width 1.02) (layer B.Cu) (net 5))
   (segment (start 173 103) (end 172 103) (width 1.02) (layer B.Cu) (net 5))
-  (segment (start 175 84) (end 175 83) (width 1.02) (layer B.Cu) (net 5))
-  (segment (start 173 86) (end 175 84) (width 1.02) (layer B.Cu) (net 5))
-  (segment (start 169 86) (end 173 86) (width 1.02) (layer B.Cu) (net 5))
+  (segment (start 161 67) (end 176 82) (width 0.81) (layer B.Cu) (net 5))
+  (segment (start 176 82) (end 176 83) (width 0.81) (layer B.Cu) (net 5))
+  (segment (start 176 84) (end 176 83) (width 1.02) (layer B.Cu) (net 5))
+  (segment (start 174 86) (end 176 84) (width 1.02) (layer B.Cu) (net 5))
+  (segment (start 169 86) (end 174 86) (width 1.02) (layer B.Cu) (net 5))
   (segment (start 167 88) (end 169 86) (width 1.02) (layer B.Cu) (net 5))
   (segment (start 167 91) (end 167 88) (width 1.02) (layer B.Cu) (net 5))
@@
   (segment (start 126 90) (end 123 93) (width 1.02) (layer B.Cu) (net 9))
   (segment (start 126 86) (end 126 90) (width 1.02) (layer B.Cu) (net 9))
-  (segment (start 169.92 80.92) (end 169.92 83) (width 1.02) (layer B.Cu) (net 10))
-  (segment (start 169 80) (end 169.92 80.92) (width 1.02) (layer B.Cu) (net 10))
+  (segment (start 170.92 81.92) (end 170.92 83) (width 1.02) (layer B.Cu) (net 10))
+  (segment (start 169 80) (end 170.92 81.92) (width 1.02) (layer B.Cu) (net 10))
+  (segment (start 155 86) (end 161 80) (width 1.02) (layer B.Cu) (net 10))
   (segment (start 161 80) (end 169 80) (width 1.02) (layer B.Cu) (net 10))
-  (segment (start 155 86) (end 161 80) (width 1.02) (layer B.Cu) (net 10))
   (segment (start 149 86) (end 155 86) (width 1.02) (layer B.Cu) (net 10))
   (segment (start 146 89) (end 149 86) (width 1.02) (layer B.Cu) (net 10))
